File: MCU/schematic/_esp8266.kicad_sch (KiCad schematic)
At the start: 20 parts, among them J1 Conn_01x06, J2 Conn_01x10, J3 Conn_01x10, SW1 SW_MEC_5G, SW2 SW_MEC_5G, U1 ESP-12F, U2 AP2112K-3.3

Commit message: Updated schematic
Connections:
- net GPIO15: now also R2.1
- net VCC: now reaches D1.2 (A)
Changed lines of the file:
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@@
+    (stroke (width 0) (type default) (color 0 0 0 0))
+  )
+  (wire (pts (xy 29.464 141.732) (xy 29.464 145.034))
     (stroke (width 0) (type default) (color 0 0 0 0))
   )
@@
   (label "GND" (at 114.3 98.806 0)
     (effects (font (size 1.27 1.27)) (justify left bottom))
+  )
+  (label "GPIO15" (at 104.902 20.574 270)
+    (effects (font (size 1.27 1.27)) (justify right bottom))
   )
   (label "EN" (at 114.3 81.026 0)
@@
     )
     (property "Datasheet" "" (id 3) (at 139.954 64.262 0)
+      (effects (font (size 1.27 1.27)) hide)
+    )
+    (pin "1")
+  )
+  (symbol (lib_id "power:VCC") (at 29.464 141.732 0) (unit 1)
+    (in_bom yes) (on_board yes) (fields_autoplaced)
+    (property "Reference" "#PWR?" (id 0) (at 29.464 145.542 0)
+      (effects (font (size 1.27 1.27)) hide)
+    )
+    (property "Value" "VCC" (id 1) (at 29.464 137.16 0))
+    (property "Footprint" "" (id 2) (at 29.464 141.732 0)
+      (effects (font (size 1.27 1.27)) hide)
+    )
+    (property "Datasheet" "" (id 3) (at 29.464 141.732 0)
       (effects (font (size 1.27 1.27)) hide)
     )
@@
       (reference "#PWR?") (unit 1) (value "GND") (footprint "")
     )
+    (path "/4cfef5ac-244f-4a84-9504-c71512519dd3"
+      (reference "#PWR?") (unit 1) (value "VCC") (footprint "")
+    )
     (path "/5893d302-71fd-4920-8b10-479a66f6de45"

Commit message: Added non-PCB files for MCU breakout board
Connections:
- net +BATT: now also J2.9 (Pin_9)
- net GND: now also J1.6 (Pin_6)
- net VCC: now also J1.4 (Pin_4), J2.8 (Pin_8)
Other:
- note added: "Note: EN = CH_PD"
Changed lines of the file:
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@@
-    (stroke (width 0) (type default) (color 0 0 0 0))
-  )
-  (wire (pts (xy 146.304 119.38) (xy 146.304 110.236))
     (stroke (width 0) (type default) (color 0 0 0 0))
   )
@@
     (stroke (width 0) (type default) (color 0 0 0 0))
   )
+  (wire (pts (xy 141.224 110.236) (xy 141.224 116.84))
+    (stroke (width 0) (type default) (color 0 0 0 0))
+  )
   (wire (pts (xy 114.3 96.266) (xy 123.444 96.266))
     (stroke (width 0) (type default) (color 0 0 0 0))
@@
     (stroke (width 0) (type default) (color 0 0 0 0))
   )
-  (wire (pts (xy 141.224 119.38) (xy 141.224 110.236))
-    (stroke (width 0) (type default) (color 0 0 0 0))
-  )
   (wire (pts (xy 114.3 86.106) (xy 123.444 86.106))
     (stroke (width 0) (type default) (color 0 0 0 0))
@@
     (stroke (width 0) (type default) (color 0 0 0 0))
   )
+  (wire (pts (xy 146.304 110.236) (xy 146.304 116.84))
+    (stroke (width 0) (type default) (color 0 0 0 0))
+  )
   (wire (pts (xy 78.994 23.114) (xy 78.994 39.878))
     (stroke (width 0) (type default) (color 0 0 0 0))
@@
     (stroke (width 0) (type default) (color 0 0 0 0))
   )
+  (text "Note: EN = CH_PD" (at 118.364 33.528 0)
+    (effects (font (size 1.27 1.27) (thickness 0.254) bold) (justify left bottom))
+  )
   (label "GPIO12" (at 165.608 45.466 180)
     (effects (font (size 1.27 1.27)) (justify right bottom))
@@
     (effects (font (size 1.27 1.27)) (justify right bottom))
   )
+  (label "Note: Pinouts not covered in tutorial" (at 110.744 43.688 0)
+    (effects (font (size 1.27 1.27) bold) (justify left bottom))
+  )
   (label "RXD" (at 165.608 37.846 180)
     (effects (font (size 1.27 1.27)) (justify right bottom))
@@
     (effects (font (size 1.27 1.27)) (justify left bottom))
   )
+  (label "VCC" (at 114.3 93.726 0)
+    (effects (font (size 1.27 1.27)) (justify left bottom))
+  )
   (label "3.3V" (at 165.608 93.726 180)
     (effects (font (size 1.27 1.27)) (justify right bottom))
@@
     (effects (font (size 1.27 1.27)) (justify right bottom))
   )
+  (label "+BATT" (at 114.3 96.266 0)
+    (effects (font (size 1.27 1.27)) (justify left bottom))
+  )
   (label "EN" (at 114.3 81.026 0)
     (effects (font (size 1.27 1.27)) (justify left bottom))
@@
   (label "EN" (at 91.948 66.802 90)
     (effects (font (size 1.27 1.27)) (justify left bottom))
+  )
+  (label "Note: ~(RST) vs. RESET" (at 114.046 26.924 0)
+    (effects (font (size 1.27 1.27) bold) (justify left bottom))
   )
   (label "GPIO16" (at 165.608 55.626 180)
@@
     (pin "6")
   )
+  (symbol (lib_id "power:VCC") (at 141.224 116.84 180) (unit 1)
+    (in_bom yes) (on_board yes) (fields_autoplaced)
+    (property "Reference" "#PWR?" (id 0) (at 141.224 113.03 0)
+      (effects (font (size 1.27 1.27)) hide)
+    )
+    (property "Value" "VCC" (id 1) (at 141.224 121.92 0))
+    (property "Footprint" "" (id 2) (at 141.224 116.84 0)
+      (effects (font (size 1.27 1.27)) hide)
+    )
+    (property "Datasheet" "" (id 3) (at 141.224 116.84 0)
+      (effects (font (size 1.27 1.27)) hide)
+    )
+    (pin "1")
+  )
   (symbol (lib_id "power:+3.3V") (at 119.38 141.732 0) (unit 1)
     (in_bom yes) (on_board yes) (fields_autoplaced)
@@
     (pin "1")
     (pin "2")
+  )
+  (symbol (lib_id "power:GND") (at 146.304 116.84 0) (unit 1)
+    (in_bom yes) (on_board yes) (fields_autoplaced)
+    (property "Reference" "#PWR?" (id 0) (at 146.304 123.19 0)
+      (effects (font (size 1.27 1.27)) hide)
+    )
+    (property "Value" "GND" (id 1) (at 146.304 121.92 0))
+    (property "Footprint" "" (id 2) (at 146.304 116.84 0)
+      (effects (font (size 1.27 1.27)) hide)
+    )
+    (property "Datasheet" "" (id 3) (at 146.304 116.84 0)
+      (effects (font (size 1.27 1.27)) hide)
+    )
+    (pin "1")
   )
   (symbol (lib_id "power:GND") (at 38.354 64.262 0) (unit 1)
@@
       (reference "#PWR?") (unit 1) (value "GND") (footprint "")
     )
+    (path "/279e0fe9-2856-4661-8b7e-8db07123bc67"
+      (reference "#PWR?") (unit 1) (value "VCC") (footprint "")
+    )
     (path "/3063ebbe-faf6-402e-a707-b52bfa8d9314"
       (reference "#PWR?") (unit 1) (value "+3.3V") (footprint "")
@@
       (reference "#PWR?") (unit 1) (value "+3.3V") (footprint "")
     )
+    (path "/74b7aaeb-8125-48bf-a6f9-6ac306b5a993"
+      (reference "#PWR?") (unit 1) (value "GND") (footprint "")
+    )
     (path "/75ccda51-ad30-411b-9a4b-c9efa31938d9"
